Commit message: updated launch

File: description/robot_core.xacro (robot description, xacro)
@@ -8,7 +8,12 @@
             </geometry>
     </xacro:property>
-    <xacro:property name="wheel_geometry">
+    <xacro:property name="wheel_geometry_v">
             <geometry>
                 <cylinder length="0.007" radius="0.016" />
+            </geometry>
+    </xacro:property>
+    <xacro:property name="wheel_geometry_c">
+            <geometry>
+                <sphere radius="0.016" />
             </geometry>
     </xacro:property>
@@ -46,9 +51,9 @@
     <link name="left_wheel">
         <visual>
-            <xacro:insert_block name="wheel_geometry"/>
+            <xacro:insert_block name="wheel_geometry_v"/>
             <material name="blue"/>
         </visual>
         <collision>
-            <xacro:insert_block name="wheel_geometry"/>
+            <xacro:insert_block name="wheel_geometry_c"/>
         </collision>
         <xacro:inertial_cylinder mass="0.1" length="0.007" radius="0.016">
@@ -65,9 +70,9 @@
     <link name="right_wheel">
         <visual>
-            <xacro:insert_block name="wheel_geometry"/>
+            <xacro:insert_block name="wheel_geometry_v"/>
             <material name="blue"/>
         </visual>
         <collision>
-            <xacro:insert_block name="wheel_geometry"/>
+            <xacro:insert_block name="wheel_geometry_c"/>
         </collision>
         <xacro:inertial_cylinder mass="0.1" length="0.007" radius="0.016">
